File: debug.sch (KiCad schematic (older format))
At the start: 13 parts, among them J1 Programmer, SW3 SW_Push, SW4 SW_Push, SW5 SW_SPDT, SW6 External RST

Commit message: Misc minor fixes
Changed lines of the file:
@@
 $EndComp
 Wire Wire Line
-	3100 1450 3300 1450
+	3150 1450 3300 1450
 $Comp
 L Device:C C?
@@
 $EndComp
 Wire Wire Line
-	3100 2400 3300 2400
+	3150 2400 3300 2400
 $Comp
 L Device:C C?
